Commit message: created a more realistic drone model

File: src/drone_kf/simple_drone.urdf (robot description, URDF)
Before this commit: robot simple_drone, 1 links, 0 joints
Links:
- added link arm_front_left, mass 0.05; collision box size=0.35 0.03 0.02; visual box size=0.35 0.03 0.02
- added link arm_front_right, mass 0.05; collision box size=0.35 0.03 0.02; visual box size=0.35 0.03 0.02
- added link arm_rear_left, mass 0.05; collision box size=0.35 0.03 0.02; visual box size=0.35 0.03 0.02
- added link arm_rear_right, mass 0.05; collision box size=0.35 0.03 0.02; visual box size=0.35 0.03 0.02
- added link camera, mass 0.05; visual box size=0.04 0.08 0.03
- added link rotor_front_left, mass 0.02; collision cylinder length=0.01 radius=0.15; visual cylinder length=0.01 radius=0.15
- added link rotor_front_right, mass 0.02; collision cylinder length=0.01 radius=0.15; visual cylinder length=0.01 radius=0.15
- added link rotor_rear_left, mass 0.02; collision cylinder length=0.01 radius=0.15; visual cylinder length=0.01 radius=0.15
- added link rotor_rear_right, mass 0.02; collision cylinder length=0.01 radius=0.15; visual cylinder length=0.01 radius=0.15
- link base_link: mass 1.0 -> 1.5; geometry collision box size=0.3 0.3 0.08; visual box size=0.3 0.3 0.08
Joints:
- added joint arm_front_left_joint: type fixed, parent base_link, child arm_front_left, origin xyz=-0.0875 0.0875 0.0 rpy=0 0 2.356194
- added joint arm_front_right_joint: type fixed, parent base_link, child arm_front_right, origin xyz=0.0875 0.0875 0.0 rpy=0 0 0.785398
- added joint arm_rear_left_joint: type fixed, parent base_link, child arm_rear_left, origin xyz=-0.0875 -0.0875 0.0 rpy=0 0 -2.356194
- added joint arm_rear_right_joint: type fixed, parent base_link, child arm_rear_right, origin xyz=0.0875 -0.0875 0.0 rpy=0 0 -0.785398
- added joint camera_joint: type fixed, parent base_link, child camera, origin xyz=0.15 0.0 -0.025 rpy=0 0.2 0
- added joint rotor_front_left_joint: type continuous, parent arm_front_left, child rotor_front_left, origin xyz=0.15 0.0 0.03 rpy=0 0 0, axis 0 0 1
- added joint rotor_front_right_joint: type continuous, parent arm_front_right, child rotor_front_right, origin xyz=0.15 0.0 0.03 rpy=0 0 0, axis 0 0 1
- added joint rotor_rear_left_joint: type continuous, parent arm_rear_left, child rotor_rear_left, origin xyz=0.15 0.0 0.03 rpy=0 0 0, axis 0 0 1
- added joint rotor_rear_right_joint: type continuous, parent arm_rear_right, child rotor_rear_right, origin xyz=0.15 0.0 0.03 rpy=0 0 0, axis 0 0 1
